Commit message: update models

File: robot_component_models/industrial_camera/model.sdf.xacro (robot description, xacro)
@@ -38,37 +38,19 @@
         </link>
     </xacro_define_macro>
-    <!--xacro_define_macro: industrial_camera_model-->
-    <xacro_define_macro name="industrial_camera_model" params="prefix update_rate horizontal_fov width height">
-        <link name="${prefix}industrial_camera">
+    <model name='simple_industrial_camera'>
+        <pose>0 0 0.2 0 0 0</pose>
+        <link name="base_link">
             <inertial>
-                <pose>0.025 0 0 0 0 0</pose>
-                <xacro_macro name="inertia_box" m="0.050" x="0.08" y="0.025" z="0.033" />
+                <xacro_macro name="inertia_box" m="0.4" x="0.4" y="0.4" z="0.4" />
             </inertial>
             <visual name="visual">
-                <xacro_macro name="geometry_mesh" uri="model://industrial_camera/meshes/industrial_camera.dae"/>
+                <xacro_macro name="geometry_box" x="0.4" y="0.4" z="0.4" />
             </visual>
             <collision name="collision">
-                <pose>0.025 0 0 0 0 0</pose>
-                <xacro_macro name="geometry_box" x="0.08" y="0.025" z="0.033" />
+                <xacro_macro name="geometry_box" x="0.4" y="0.4" z="0.4" />
             </collision>
-            <sensor name="${prefix}industrial_camera" type="camera">
-                <always_on>1</always_on>
-                <update_rate>${update_rate}</update_rate>
-                <camera>
-                    <horizontal_fov>${horizontal_fov}</horizontal_fov>
-                    <image>
-                        <width>${width}</width>
-                        <height>${height}</height>
-                    </image>
-                    <clip>
-                        <near>0.1</near>
-                        <far>100</far>
-                    </clip>
-                </camera>
-            </sensor>
         </link>
-    </xacro_define_macro>
-    <model name='simple_industrial_camera'>
-        <xacro_macro name="industrial_camera_model" prefix="simple_" update_rate="30" horizontal_fov="1" width="640" height="480"/>
+        <xacro_macro name="industrial_camera" prefix="simple_" parent="base_link" pose="0 0 0.216 0 0 0"
+                update_rate="30" horizontal_fov="1" width="640" height="480"/>
     </model>
 </sdf>

File: robot_component_models/rplidar_a2/model.sdf.xacro (robot description, xacro)
@@ -48,50 +48,21 @@
         </link>
     </xacro_define_macro>
-    <!--xacro_define_macro: rplidar_a2_model-->
-    <xacro_define_macro name="rplidar_a2_model" params="prefix update_rate samples visualize">
-        <link name="${prefix}rplidar_a2">
+    <!--rplidar a2-->
+    <model name='simple_rplidar_a2'>
+        <pose>0 0 0.2 0 0 0</pose>
+        <link name="base_link">
             <inertial>
-                <pose>0 0 0.02 0 0 0</pose>
-                <xacro_macro name="inertia_cylinder" m="0.005" r="0.04" l="0.04" />
+                <xacro_macro name="inertia_box" m="0.4" x="0.4" y="0.4" z="0.4" />
             </inertial>
             <visual name="visual">
-                <xacro_macro name="geometry_mesh" uri="model://rplidar_a2/meshes/rplidar_a2.dae"/>
+                <xacro_macro name="geometry_box" x="0.4" y="0.4" z="0.4" />
             </visual>
             <collision name="collision">
-                <pose>0 0 0.02 0 0 0</pose>
-                <xacro_macro name="geometry_cylinder" r="0.04" l="0.04"/>
+                <xacro_macro name="geometry_box" x="0.4" y="0.4" z="0.4" />
             </collision>
-            <sensor name="${prefix}rplidar_a2" type="gpu_lidar">
-                <pose>0 0 0.03 0 0 0</pose>
-                <always_on>true</always_on>
-                <visualize>${visualize}</visualize>
-                <update_rate>${update_rate}</update_rate>
-                <ray>
-                    <scan>
-                        <horizontal>
-                            <samples>${samples}</samples>
-                            <resolution>0.9</resolution>
-                            <min_angle>-3.14159265359</min_angle>
-                            <max_angle>3.14159265359</max_angle>
-                        </horizontal>
-                    </scan>
-                    <range>
-                        <min>0.15</min>
-                        <max>12.0</max>
-                    </range>
-                </ray>
-                <noise>
-                    <type>gaussian</type>
-                    <mean>0.0</mean>
-                    <stddev>0.01</stddev>
-                </noise>
-            </sensor>
         </link>
-    </xacro_define_macro>
-    <!--rplidar a2-->
-    <model name='simple_rplidar_a2'>
         <!--update_rate(10-15),samples(400)-->
-        <pose>0 0 0.1 0 0 0</pose>
-        <xacro_macro name="rplidar_a2" prefix="simple_" update_rate="10" samples="400" visualize="true"/>
+        <xacro_macro name="rplidar_a2" prefix="simple_"  parent="base_link" pose="0 0 0.2 0 0 0"
+            update_rate="10" samples="400" visualize="true"/>
     </model>
 </sdf>

File: robot_models/rmua19_standard_robot/model.sdf.xacro (robot description, xacro)
@@ -4,12 +4,14 @@
     <xacro_include_definition uri="model://rplidar_a2/model.sdf.xacro" />
     <xacro_include_definition uri="model://industrial_camera/model.sdf.xacro" />
+    <xacro_include_definition uri="model://rm21_armor_module/model.sdf.xacro" />
+    <xacro_include_definition uri="model://rm21_light_indicator_module/model.sdf.xacro" />
+    <xacro_include_definition uri="model://rm21_speed_monitor_module/model.sdf.xacro" />
     <xacro_include_definition uri="file://chassis_wheel.def.xacro" />
-    <xacro_include_definition uri="file://referee_system.def.xacro" />
     <!--property defination-->
-    <xacro_define_property name="chassis_mass" value="10.0" />
+    <xacro_define_property name="chassis_mass" value="15.0" />
     <!-- <xacro_define_property name="wheel_offset_x" value="0.207571" /> -->
     <!-- <xacro_define_property name="wheel_offset_y" value="0.194019" /> -->
-    <xacro_define_property name="gimbal_yaw_mass" value="0.5" />
-    <xacro_define_property name="gimbal_pitch_mass" value="0.2" />
+    <xacro_define_property name="gimbal_yaw_mass" value="1.0" />
+    <xacro_define_property name="gimbal_pitch_mass" value="0.5" />
     <xacro_define_property name="light_bar_rgb" value="1 1 1" />
     <!--macro defination: rmua19_standard_robot_base-->
@@ -45,6 +47,4 @@
             </sensor>
         </link>
-        <!--light_indicator-->
-        <xacro_macro name="light_indicator" prefix="" parent="chassis" rgb="${light_bar_rgb}" pose="-0.207 0 0.1 0 0 0"/>
         <!--front_left wheel link and joint-->
         <xacro_macro name="chassis_wheel_l"  prefix="front_left" parent="chassis" pose="0.207 0.194 0 0 0 0"/>
@@ -55,13 +55,4 @@
         <!--rear_right wheel link and joint-->
         <xacro_macro name="chassis_wheel_l"  prefix="rear_right" parent="chassis" pose="-0.207 -0.194 0 0 0 0"/>
-        <!--4 armors -->
-        <!--front armors -->
-        <xacro_macro name="armor" suffix="_0" parent="chassis" rgb="${light_bar_rgb}" x="0.197" y="0" z="0.061" yaw="0"/>
-        <!--rear armors -->
-        <xacro_macro name="armor" suffix="_2" parent="chassis" rgb="${light_bar_rgb}" x="-0.197" y="0" z="0.061" yaw="3.14159"/>
-        <!--left armors -->
-        <xacro_macro name="armor" suffix="_1" parent="chassis" rgb="${light_bar_rgb}" x="0" y="0.116" z="0.060" yaw="1.5708"/>
-        <!--right armors -->
-        <xacro_macro name="armor" suffix="_3" parent="chassis" rgb="${light_bar_rgb}" x="0" y="-0.116" z="0.060" yaw="-1.5708"/>
         <!--gimbal yaw module-->
         <joint name="gimbal_yaw_joint" type="revolute">
@@ -102,5 +93,5 @@
             <pose relative_to="gimbal_pitch_joint">0 0 0 0 0 0</pose>
             <inertial>
-                <pose>0.05 0 0 0 0 0</pose>
+                <pose>0.02 0 0 0 0 0</pose>
                 <xacro_macro name="inertia_box"  m="${gimbal_pitch_mass}" x="0.25" y="0.09" z="0.10" />
             </inertial>
@@ -108,4 +99,19 @@
                     uri="model://rmua19_standard_robot/meshes/gimbal_pitch.dae"/>
         </link>
+        <!--for referee system -->
+        <!--front armors -->
+        <xacro_macro name="small_armor_with_support" suffix="_0" parent="chassis"
+                rgb="${light_bar_rgb}" pose="0.197 0 0.061 0 0 0"/>
+        <!--left armors -->
+        <xacro_macro name="small_armor_with_support" suffix="_1" parent="chassis"
+                rgb="${light_bar_rgb}" pose="0 0.116 0.061 0 0 1.5708"/>
+        <!--rear armors -->
+        <xacro_macro name="small_armor_with_support" suffix="_2" parent="chassis"
+                rgb="${light_bar_rgb}" pose="-0.197 0 0.061 0 0 3.14"/>
+        <!--right armors -->
+        <xacro_macro name="small_armor_with_support" suffix="_3" parent="chassis"
+                rgb="${light_bar_rgb}" pose="0 -0.116 0.061 0 0 -1.5708"/>
+        <!--light_indicator-->
+        <xacro_macro name="light_indicator" prefix="" parent="chassis" rgb="${light_bar_rgb}" pose="-0.207 0 0.1 0 0 0"/>
         <!--speed_monitor_17mm-->
         <xacro_macro name="speed_monitor_17mm" prefix="" parent="gimbal_pitch" rgb="${light_bar_rgb}" pose="0.07 0 0 0 0 0"/>
