Commit message: update model sdf style

File: models/rm21_armor_module/model.sdf.xacro (robot description, xacro)
@@ -1,147 +1,8 @@
 <?xml version="1.0"?>
 <sdf version="1.7">
+    <!--include defination-->
+    <xacro_include_definition uri="model://rm21_armor_module/rm21_armor_module.def.xacro" />
     <!--property defination-->
     <xacro_define_property name="global_armor_sticker_map_uri" value="model://rm21_armor_module/materials/textures/armor_sticker_num1.png" />
-    <!--macro defination: small armor module-->
-    <xacro_define_macro name="small_armor" params="suffix parent rgb sticker_uri pose">
-        <joint name="small_armor${suffix}_joint" type="fixed">
-            <pose relative_to="${parent}">${pose}</pose>
-            <parent>${parent}</parent>
-            <child>small_armor${suffix}</child>
-        </joint>
-        <link name="small_armor${suffix}">
-            <pose relative_to="small_armor${suffix}_joint">0 0 0 0 0 0</pose>
-            <inertial>
-                <pose>0 0 0.065 0 0 0</pose>
-                <xacro_macro name="inertia_box"  m="0.1" x="0.012" y="0.141" z="0.13"/>
-            </inertial>
-            <visual name="visual">
-                <xacro_macro name="geometry_mesh" uri="model://rm21_armor_module/meshes/small_armor.dae"/>
-            </visual>
-            <visual name="target_visual">
-                <xacro_macro name="geometry_mesh" uri="model://rm21_armor_module/meshes/small_armor_target.dae"/>
-            </visual>
-            <visual name="light_bar_visual">
-                <xacro_macro name="geometry_mesh" uri="model://rm21_armor_module/meshes/small_armor_light_bar.dae"/>
-                <material>
-                    <ambient>${rgb} 1</ambient>
-                    <diffuse>${rgb} 1</diffuse>
-                    <specular>1 1 1 1</specular>
-                    <emissive>${rgb} 1</emissive>
-                </material>
-            </visual>
-            <visual name="sticker_visual">
-                <pose>0.014 0 0.065 1.5708 0 1.5708</pose>
-                <geometry>
-                    <plane>
-                        <normal>0 0 1</normal>
-                        <size>0.1 0.1</size>
-                    </plane>
-                </geometry>
-                <material>
-                    <diffuse>1.0 1.0 1.0</diffuse>
-                    <specular>1.0 1.0 1.0</specular>
-                    <ambient>1.0 1.0 1.0</ambient>
-                    <pbr>
-                        <metal>
-                            <albedo_map>${sticker_uri}</albedo_map>
-                        </metal>
-                    </pbr>
-                </material>
-            </visual>
-            <collision name="collision">
-                <xacro_macro name="geometry_mesh" uri="model://rm21_armor_module/meshes/small_armor.dae"/>
-            </collision>
-            <collision name="target_collision">
-                <xacro_macro name="geometry_mesh" uri="model://rm21_armor_module/meshes/small_armor_target.dae"/>
-            </collision>
-        </link>
-    </xacro_define_macro>
-    <!--macro defination: large armor module-->
-    <xacro_define_macro name="large_armor" params="suffix parent rgb sticker_uri pose">
-        <joint name="large_armor${suffix}_joint" type="fixed">
-            <pose relative_to="${parent}">${pose}</pose>
-            <parent>${parent}</parent>
-            <child>large_armor${suffix}</child>
-        </joint>
-        <link name="large_armor${suffix}">
-            <pose relative_to="large_armor${suffix}_joint">0 0 0 0 0 0</pose>
-            <inertial>
-                <pose>0 0 0.065 0 0 0</pose>
-                <xacro_macro name="inertia_box"  m="0.1" x="0.012" y="0.141" z="0.13"/>
-            </inertial>
-            <visual name="visual">
-                <xacro_macro name="geometry_mesh" uri="model://rm21_armor_module/meshes/large_armor.dae"/>
-            </visual>
-            <visual name="target_visual">
-                <xacro_macro name="geometry_mesh" uri="model://rm21_armor_module/meshes/large_armor_target.dae"/>
-            </visual>
-            <visual name="light_bar_visual">
-                <xacro_macro name="geometry_mesh" uri="model://rm21_armor_module/meshes/large_armor_light_bar.dae"/>
-                <material>
-                    <ambient>${rgb} 1</ambient>
-                    <diffuse>${rgb} 1</diffuse>
-                    <specular>1 1 1 1</specular>
-                    <emissive>${rgb} 1</emissive>
-                </material>
-            </visual>
-            <visual name="sticker_visual">
-                <pose>0.014 0 0.065 1.5708 0 1.5708</pose>
-                <geometry>
-                    <plane>
-                        <normal>0 0 1</normal>
-                        <size>0.1 0.1</size>
-                    </plane>
-                </geometry>
-                <material>
-                    <diffuse>1.0 1.0 1.0</diffuse>
-                    <specular>1.0 1.0 1.0</specular>
-                    <ambient>1.0 1.0 1.0</ambient>
-                    <pbr>
-                        <metal>
-                            <albedo_map>${sticker_uri}</albedo_map>
-                        </metal>
-                    </pbr>
-                </material>
-            </visual>
-            <collision name="collision">
-                <xacro_macro name="geometry_mesh" uri="model://rm21_armor_module/meshes/large_armor.dae"/>
-            </collision>
-            <collision name="target_collision">
-                <xacro_macro name="geometry_mesh" uri="model://rm21_armor_module/meshes/large_armor_target.dae"/>
-            </collision>
-        </link>
-    </xacro_define_macro>
-    <!--macro defination: armor support frame-->
-    <xacro_define_macro name="armor_support_frame" params="suffix parent pose">
-        <joint name="armor_support_frame${suffix}_joint" type="fixed">
-            <pose relative_to="${parent}">${pose}</pose>
-            <parent>${parent}</parent>
-            <child>armor_support_frame${suffix}</child>
-        </joint>
-        <link name="armor_support_frame${suffix}">
-            <pose relative_to="armor_support_frame${suffix}_joint">0 0 0 0 0 0</pose>
-            <inertial>
-                <pose>0.035 0 0 0 0 0</pose>
-                <xacro_macro name="inertia_box"  m="0.1" x="0.071" y="0.111" z="0.124"/>
-            </inertial>
-            <visual name="visual">
-                <xacro_macro name="geometry_mesh" uri="model://rm21_armor_module/meshes/armor_support_frame.dae"/>
-            </visual>
-            <collision name="collision">
-                <xacro_macro name="geometry_mesh" uri="model://rm21_armor_module/meshes/armor_support_frame.dae"/>
-            </collision>
-        </link>
-    </xacro_define_macro>
-    <!--macro defination: small armor module with support frame-->
-    <xacro_define_macro name="small_armor_with_support" params="suffix parent rgb sticker_uri pose">
-        <xacro_macro name="armor_support_frame" suffix="${suffix}" parent="${parent}" pose="${pose}"/>
-        <xacro_macro name="small_armor" suffix="${suffix}" parent="armor_support_frame${suffix}" rgb="${rgb}" sticker_uri="${sticker_uri}" pose="0.075 0 -0.071 0 -0.262 0"/>
-    </xacro_define_macro>
-    <!--macro defination: large armor module with support frame-->
-    <xacro_define_macro name="large_armor_with_support" params="suffix parent rgb sticker_uri pose">
-        <xacro_macro name="armor_support_frame" suffix="${suffix}" parent="${parent}" pose="${pose}"/>
-        <xacro_macro name="large_armor" suffix="${suffix}" parent="armor_support_frame${suffix}" rgb="${rgb}" sticker_uri="${sticker_uri}" pose="0.075 0 -0.071 0 -0.262 0"/>
-    </xacro_define_macro>
     <!--rm21_armor_module example-->
     <model name='rm21_armor_module'>

File: models/rm21_light_indicator_module/model.sdf.xacro (robot description, xacro)
@@ -1,35 +1,6 @@
 <?xml version="1.0"?>
 <sdf version="1.7">
-    <!--macro defination: light indicator module-->
-    <xacro_define_macro name="light_indicator" params="prefix parent rgb pose">
-        <joint name="${prefix}light_indicator_joint" type="fixed">
-            <pose relative_to="${parent}">${pose}</pose>
-            <parent>${parent}</parent>
-            <child>${prefix}light_indicator</child>
-        </joint>
-        <link name="${prefix}light_indicator">
-            <pose relative_to="${prefix}light_indicator_joint">0 0 0 0 0 0</pose>
-            <inertial>
-                <pose>0 0 0.04 0 0 0</pose>
-                <xacro_macro name="inertia_box" m="0.1" x="0.05" y="0.28" z="0.04"/>
-            </inertial>
-            <visual name="light_indicator_holder_visual">
-                <xacro_macro name="geometry_mesh" uri="model://rm21_light_indicator_module/meshes/light_indicator_holder.dae"/>
-            </visual>
-            <visual name="light_indicator_bar_visual">
-                <xacro_macro name="geometry_mesh" uri="model://rm21_light_indicator_module/meshes/light_indicator_bar.dae"/>
-                <material>
-                    <ambient>${rgb} 1</ambient>
-                    <diffuse>${rgb} 1</diffuse>
-                    <specular>1 1 1 1</specular>
-                    <emissive>${rgb} 1</emissive>
-                </material>
-            </visual>
-            <collision name="light_indicator_bar_collision">
-                <pose>0 0 0.06 0 0 0</pose>
-                <xacro_macro name="geometry_box" x="0.05" y="0.28" z="0.04"/>
-            </collision>
-        </link>
-    </xacro_define_macro>
+     <!--include defination-->
+    <xacro_include_definition uri="model://rm21_light_indicator_module/rm21_light_indicator_module.def.xacro" />
     <!--rm21_light_indicator_module example-->
     <model name='rm21_light_indicator_module'>
@@ -46,5 +17,5 @@
             </collision>
         </link>
-        <xacro_macro name="light_indicator" prefix="" parent="base_link" rgb="1 0 0" pose="0 0 0.2 0 0 0"/>
+        <xacro_macro name="light_indicator" suffix="" parent="base_link" rgb="1 0 0" pose="0 0 0.2 0 0 0"/>
     </model>
 </sdf>

File: models/rm21_speed_monitor_module/model.sdf.xacro (robot description, xacro)
@@ -1,35 +1,6 @@
 <?xml version="1.0"?>
 <sdf version="1.7">
-    <!--macro defination: speed monitor 17mm module-->
-    <xacro_define_macro name="speed_monitor_17mm" params="prefix parent rgb pose">
-        <joint name="${prefix}speed_monitor_17mm_joint" type="fixed">
-            <pose relative_to="${parent}">${pose}</pose>
-            <parent>${parent}</parent>
-            <child>${prefix}speed_monitor_17mm</child>
-        </joint>
-        <link name="${prefix}speed_monitor_17mm">
-            <pose relative_to="${prefix}speed_monitor_17mm_joint">0 0 0 0 0 0</pose>
-            <inertial>
-                <pose>0.055 0 0 0 0 0</pose>
-                <xacro_macro name="inertia_box" m="0.1" x="0.11" y="0.043" z="0.041"/>
-            </inertial>
-            <visual name="visual">
-                <xacro_macro name="geometry_mesh" uri="model://rm21_speed_monitor_module/meshes/speed_monitor_17mm.dae"/>
-            </visual>
-            <visual name="light_bar_visual">
-                <xacro_macro name="geometry_mesh" uri="model://rm21_speed_monitor_module/meshes/speed_monitor_17mm_light_bar.dae"/>
-                <material>
-                    <ambient>${rgb} 1</ambient>
-                    <diffuse>${rgb} 1</diffuse>
-                    <specular>1 1 1 1</specular>
-                    <emissive>${rgb} 1</emissive>
-                </material>
-            </visual>
-            <collision name="collision">
-                <pose>0.055 0 0 0 0 0</pose>
-                <xacro_macro name="geometry_box" x="0.11" y="0.043" z="0.041"/>
-            </collision>
-        </link>
-    </xacro_define_macro>
+     <!--include defination-->
+    <xacro_include_definition uri="model://rm21_speed_monitor_module/rm21_speed_monitor_module.def.xacro" />
     <!--rm21_speed_monitor_module example-->
     <model name='rm21_speed_monitor_module'>
@@ -46,5 +17,5 @@
             </collision>
         </link>
-        <xacro_macro name="speed_monitor_17mm" prefix="my_" parent="base_link" rgb="1 0 0" pose="0.2 0 0 0 0 0"/>
+        <xacro_macro name="speed_monitor_17mm" suffix="_1" parent="base_link" rgb="1 0 0" pose="0.2 0 0 0 0 0"/>
     </model>
 </sdf>

File: models/rm_fluorescent_projectile_17mm/model.sdf.xacro (robot description, xacro)
@@ -3,25 +3,7 @@
     <xacro_define_property name="projectile_r" value="0.0084" />
     <xacro_define_property name="projectile_m" value="0.0032" />
-    <xacro_define_macro name="rm_fluorescent_projectile" params="suffix m r">
-        <link name ='rm_projectile${suffix}'>
-            <inertial>
-                <xacro_macro name="inertia_sphere"  m="${m}" r="${r}"/>
-            </inertial>
-            <visual name ='visual'>
-                <xacro_macro name="geometry_sphere" r="${r}"/>
-                <material>
-                    <ambient>0 0.6 0 1</ambient>
-                    <diffuse>0 0.6 0 1</diffuse>
-                    <specular>1 1 1 1</specular>
-                    <emissive>0 0.6 0 1 1</emissive>
-                </material>
-            </visual>
-            <collision name ='collision'>
-                <xacro_macro name="geometry_sphere" r="${r}"/>
-            </collision>
-        </link>
-    </xacro_define_macro>
+    <xacro_include_definition uri="model://rm_fluorescent_projectile_17mm/rm_fluorescent_projectile.def.xacro"/>
     <model name="rm_projectile_17mm">
-        <xacro_macro name="rm_fluorescent_projectile" suffix="_17mm" m="${projectile_m}" r="${projectile_r}"/>
+        <xacro_macro name="rm_fluorescent_projectile" m="${projectile_m}" r="${projectile_r}"/>
     </model>
 </sdf>

File: models/rm_fluorescent_projectile_42mm/model.sdf.xacro (robot description, xacro)
@@ -3,7 +3,7 @@
     <xacro_define_property name="projectile_r" value="0.021" />
     <xacro_define_property name="projectile_m" value="0.041" />
-    <xacro_include_definition uri="model://rm_fluorescent_projectile_17mm/model.sdf.xacro"/>
+    <xacro_include_definition uri="model://rm_fluorescent_projectile_17mm/rm_fluorescent_projectile.def.xacro"/>
     <model name="rm_projectile_42mm">
-        <xacro_macro name="rm_fluorescent_projectile" suffix="_42mm" m="${projectile_m}" r="${projectile_r}"/>
+        <xacro_macro name="rm_fluorescent_projectile" m="${projectile_m}" r="${projectile_r}"/>
     </model>
 </sdf>

File: models/rm_projectile_17mm/model.sdf.xacro (robot description, xacro)
@@ -3,19 +3,7 @@
     <xacro_define_property name="projectile_r" value="0.0084" />
     <xacro_define_property name="projectile_m" value="0.0032" />
-    <xacro_define_macro name="rm_projectile" params="suffix m r">
-        <link name ='rm_projectile${suffix}'>
-            <inertial>
-                <xacro_macro name="inertia_sphere"  m="${m}" r="${r}"/>
-            </inertial>
-            <visual name ='visual'>
-                <xacro_macro name="geometry_sphere" r="${r}"/>
-            </visual>
-            <collision name ='collision'>
-                <xacro_macro name="geometry_sphere" r="${r}"/>
-            </collision>
-        </link>
-    </xacro_define_macro>
+    <xacro_include_definition uri="model://rm_projectile_17mm/rm_projectile.def.xacro"/>
     <model name="rm_projectile_17mm">
-        <xacro_macro name="rm_projectile" suffix="_17mm" m="${projectile_m}" r="${projectile_r}"/>
+        <xacro_macro name="rm_projectile" m="${projectile_m}" r="${projectile_r}"/>
     </model>
 </sdf>

File: models/rm_projectile_42mm/model.sdf.xacro (robot description, xacro)
@@ -3,7 +3,7 @@
     <xacro_define_property name="projectile_r" value="0.021" />
     <xacro_define_property name="projectile_m" value="0.041" />
-    <xacro_include_definition uri="model://rm_projectile_17mm/model.sdf.xacro" />
+    <xacro_include_definition uri="model://rm_projectile_17mm/rm_projectile.def.xacro"/>
     <model name="rm_projectile_42mm">
-        <xacro_macro name="rm_projectile" suffix="_42mm" m="${projectile_m}" r="${projectile_r}"/>
+        <xacro_macro name="rm_projectile" m="${projectile_m}" r="${projectile_r}"/>
     </model>
 </sdf>
