Commit message: simplify the collision of robot model

File: models/rm21_armor_module/rm21_armor_module.def.xacro (robot description, xacro)
@@ -12,5 +12,5 @@
             <inertial>
                 <pose>0 0 0.065 0 0 0</pose>
-                <xacro_macro name="inertia_box"  m="0.1" x="0.012" y="0.141" z="0.13"/>
+                <xacro_macro name="inertia_box"  m="0.1" x="0.0127" y="0.141" z="0.13"/>
             </inertial>
             <visual name="visual">
@@ -49,5 +49,6 @@
             </visual>
             <collision name="collision">
-                <xacro_macro name="geometry_mesh" uri="model://rm21_armor_module/meshes/small_armor.dae"/>
+                <pose>0 0 0.065 0 0 0</pose>
+                <xacro_macro name="geometry_box" x="0.0127" y="0.141" z="0.13"/>
             </collision>
             <collision name="target_collision">
@@ -67,5 +68,5 @@
             <inertial>
                 <pose>0 0 0.065 0 0 0</pose>
-                <xacro_macro name="inertia_box"  m="0.1" x="0.012" y="0.141" z="0.13"/>
+                <xacro_macro name="inertia_box"  m="0.1" x="0.012" y="0.236" z="0.13"/>
             </inertial>
             <visual name="visual">
@@ -104,5 +105,6 @@
             </visual>
             <collision name="collision">
-                <xacro_macro name="geometry_mesh" uri="model://rm21_armor_module/meshes/large_armor.dae"/>
+                <pose>0 0 0.065 0 0 0</pose>
+                <xacro_macro name="geometry_box" x="0.012" y="0.236" z="0.13"/>
             </collision>
             <collision name="target_collision">
@@ -128,5 +130,6 @@
             </visual>
             <collision name="collision">
-                <xacro_macro name="geometry_mesh" uri="model://rm21_armor_module/meshes/armor_support_frame.dae"/>
+                <pose>0.015 0 0 0 0 0</pose>
+                <xacro_macro name="geometry_box" x="0.03" y="0.11" z="0.08"/>
             </collision>
         </link>

File: models/rmua19_standard_robot/rmua19_standard_robot.def.xacro (robot description, xacro)
@@ -69,5 +69,11 @@
                 <xacro_macro name="inertia_cylinder"  m="${global_gimbal_yaw_mass}" r="0.05" l="0.17"/>
             </inertial>
-            <xacro_macro name="visual_collision_with_mesh" prefix="gimbal_yaw" uri="model://rmua19_standard_robot/meshes/gimbal_yaw.dae"/>
+            <visual name="visual">
+                <xacro_macro name="geometry_mesh" uri="model://rmua19_standard_robot/meshes/gimbal_yaw.dae"/>
+            </visual>
+            <collision name="collision">
+                <pose>0 0 0.0885 0 0 0</pose>
+                <xacro_macro name="geometry_box" x="0.065" y="0.117" z="0.177"/>
+            </collision>
         </link>
         <!--gimbal pitch module-->
@@ -90,5 +96,15 @@
                 <xacro_macro name="inertia_box"  m="${global_gimbal_pitch_mass}" x="0.25" y="0.09" z="0.10" />
             </inertial>
-            <xacro_macro name="visual_collision_with_mesh" prefix="gimbal_pitch" uri="model://rmua19_standard_robot/meshes/gimbal_pitch.dae"/>
+            <visual name="visual">
+                <xacro_macro name="geometry_mesh" uri="model://rmua19_standard_robot/meshes/gimbal_pitch.dae"/>
+            </visual>
+            <collision name="collision_main">
+                <pose>0.015 0 0 0 0 0</pose>
+                <xacro_macro name="geometry_box"  x="0.1" y="0.0915" z="0.08"/>
+            </collision>
+            <collision name="collision_box">
+                <pose>-0.011 0 0.043 0 0 0</pose>
+                <xacro_macro name="geometry_box"  x="0.14801" y="0.07" z="0.065"/>
+            </collision>
         </link>
         <!--for referee system -->
